File: stemma-mach32.kicad_pcb (KiCad board)
At the start: 2 copper layers, 17.8 x 35.6 mm, 32 parts, among them J1 Conn_01x09_Male, J2 Conn_01x04_Male, J3 Conn_01x04_Male, J4 Conn_01x09_Male, J5 DebugEdge_02x04, Q1 BSS138, Q2 BSS138, U1 AP2112K-3.3, U2 MACHXO2-32QFN

Commit message: fix: correct the FPGA package and DebugEdge schematic connections
Use the manufacturer's exact HC SG32 ordering and pinout data. Restore the schematic-to-PCB mapping broken by stale label placement around the pinned DebugEdge symbol, preserving copper and submodule revisions. Version the legacy symbol cache and retain all upstream licence scopes.
Parts:
- FB1: value Ferrite_Bead_Small -> 30Ω@100MHz
Changed lines of the file:
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@@
       (effects (font (size 1 1) (thickness 0.15)))
     )
-    (fp_text value Ferrite_Bead_Small (at 0 1.43) (layer F.Fab)
+    (fp_text value "30Ω@100MHz" (at 0 1.43) (layer F.Fab)
       (effects (font (size 1 1) (thickness 0.15)))
     )
